Commit message: wander: 4-direction check, urdf laser_yaw=pi

File: src/scr_description/urdf/ugv02.urdf.xacro (robot description, xacro)
@@ -23,5 +23,5 @@
   <xacro:property name="laser_y"   value="0.0"/>   <!-- ★ 왼(+)/오른(-) -->
   <xacro:property name="laser_z"   value="0.090"/> <!-- ★ base_link 원점(바퀴 축 높이)에서 라이다 스캔 면까지 높이 -->
-  <xacro:property name="laser_yaw" value="0.0"/>   <!-- ★ 라이다 0° 방향. RPLIDAR 는 0°가 로봇 뒤쪽인 경우가 있음 → 앞에 물건 두고 RViz 에서 확인, 반대면 ${pi} -->
+  <xacro:property name="laser_yaw" value="${pi}"/> <!-- ✅ 10-29 실측: 로봇 앞 물체가 라이다 +178° 로 찍힘 → 0°가 로봇 뒤쪽 → pi (wander.py --check) -->
   <!-- ===== 부품 ===== -->
   <!-- 바닥에 찍힌 로봇 중심점. Nav2·브리지 odom 의 기준 -->

Commit message: wander: stop 0.55m, min turn 1.5s, clean Ctrl+C

File: src/scr_description/urdf/ugv02.urdf.xacro (robot description, xacro)
@@ -23,5 +23,5 @@
   <xacro:property name="laser_y"   value="0.0"/>   <!-- ★ 왼(+)/오른(-) -->
   <xacro:property name="laser_z"   value="0.090"/> <!-- ★ base_link 원점(바퀴 축 높이)에서 라이다 스캔 면까지 높이 -->
-  <xacro:property name="laser_yaw" value="${pi}"/> <!-- ✅ 10-29 실측: 로봇 앞 물체가 라이다 +178° 로 찍힘 → 0°가 로봇 뒤쪽 → pi (wander.py --check) -->
+  <xacro:property name="laser_yaw" value="${pi}"/> <!-- ✅ 10-29 실측: 로봇 앞 물체가 라이다 +178° 로 찍힘 → 0°가 로봇 뒤쪽 → pi (wander.py check) -->
   <!-- ===== 부품 ===== -->
   <!-- 바닥에 찍힌 로봇 중심점. Nav2·브리지 odom 의 기준 -->

Commit message: Real odom calibration: wheels inflate yaw 2.3-2.7x, gyro within 5%; track 0.40 fixes wall overlap

File: src/scr_description/urdf/ugv02.urdf.xacro (robot description, xacro)
@@ -13,7 +13,7 @@
   <xacro:property name="width"         value="0.230"/>  <!-- 좌우 폭, 바퀴 포함 (스펙) -->
   <xacro:property name="height"        value="0.094"/>  <!-- 바닥 ~ 차체 윗면 (스펙) -->
-  <xacro:property name="wheel_radius"  value="0.040"/>  <!-- ★ 바퀴 반지름 -->
+  <xacro:property name="wheel_radius"  value="0.0375"/> <!-- 실측 10-31: 지름 7.5 cm -->
   <xacro:property name="wheel_width"   value="0.035"/>  <!-- ★ 바퀴 폭 -->
-  <xacro:property name="track_width"   value="0.160"/>  <!-- ★ 좌우 바퀴 중심 간격. 브리지 track_width 파라미터와 같은 뜻 (odom 보정으로 실제 유효값은 따로 구함) -->
+  <xacro:property name="track_width"   value="0.170"/>  <!-- 실측 10-31: 좌우 가운데 바퀴 중심 간격 17 cm. 브리지 track_width 파라미터와 같은 뜻 (odom 보정으로 실제 유효값은 따로 구함) -->
   <xacro:property name="wheel_base"    value="0.170"/>  <!-- ★ 맨 앞 바퀴 ~ 맨 뒤 바퀴 중심 거리 -->
   <xacro:property name="body_width"    value="${width - 2 * wheel_width}"/>
@@ -22,5 +22,6 @@
   <xacro:property name="laser_x"   value="0.0"/>   <!-- ★ 앞(+)/뒤(-) -->
   <xacro:property name="laser_y"   value="0.0"/>   <!-- ★ 왼(+)/오른(-) -->
-  <xacro:property name="laser_z"   value="0.090"/> <!-- ★ base_link 원점(바퀴 축 높이)에서 라이다 스캔 면까지 높이 -->
+  <xacro:property name="laser_scan_height" value="0.195"/> <!-- 실측 10-31: 바닥 ~ 라이다 창 가운데 19.5 cm. 이 높이 아래 물체(의자 다리 등)는 라이다가 못 봄 -->
+  <xacro:property name="laser_z"   value="${laser_scan_height - wheel_radius}"/> <!-- base_link 원점(바퀴 축 높이) 기준. wheel_radius 가 ★ 라 이 값도 바퀴 실측 후 확정 -->
   <xacro:property name="laser_yaw" value="${pi}"/> <!-- ✅ 10-29 실측: 로봇 앞 물체가 라이다 +178° 로 찍힘 → 0°가 로봇 뒤쪽 → pi (wander.py check) -->
   <!-- ===== 부품 ===== -->
